File: Keyboard-Saturn.kicad_pcb (KiCad board)
At the start: 2 copper layers, 438.9 x 124.3 mm, 215 parts, among them J1 OLED_128x32, SW1 SW_Push, SW10 SW_Push, SW11 SW_Push, SW12 SW_Push, SW13 SW_Push, SW14 SW_Push, SW15 SW_Push, SW16 SW_Push, SW17 SW_Push, SW18 SW_Push, SW19 SW_Push, SW2 SW_Push, SW20 SW_Push, SW21 SW_Push, SW22 SW_Push, SW23 SW_Push, SW24 SW_Push, SW25 SW_Push, SW26 SW_Push, SW27 SW_Push, SW28 SW_Push, SW29 SW_Push, SW3 SW_Push, SW30 SW_Push, SW31 SW_Push, SW32 SW_Push, SW33 SW_Push, SW34 SW_Push, SW35 SW_Push, SW36 SW_Push, SW37 SW_Push, SW38 SW_Push, SW39 SW_Push, SW4 SW_Push, SW40 SW_Push, SW41 SW_Push, SW42 SW_Push, SW43 SW_Push, SW44 SW_Push, SW45 SW_Push, SW46 SW_Push, SW47 SW_Push, SW48 SW_Push, SW49 SW_Push, SW5 SW_Push, SW50 SW_Push, SW51 SW_Push, SW52 SW_Push, SW53 SW_Push, SW54 SW_Push, SW55 SW_Push, SW56 SW_Push, SW57 SW_Push, SW58 SW_Push, SW59 SW_Push, SW6 SW_Push, SW60 SW_Push, SW61 SW_Push, SW62 SW_Push, SW63 SW_Push, SW64 Rctrl, SW65 SW_Push, SW66 SW_Push, SW67 SW_Push, SW68 SW_Push, SW69 SW_Push, SW7 SW_Push, SW70 SW_Push, SW71 SW_Push, SW72 SW_Push, SW73 SW_Push, SW74 SW_Push, SW75 SW_Push, SW77 SW_Push, SW78 SW_Push, SW79 SW_Push, SW8 SW_Push, SW80 SW_Push, SW81 SW_Push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

Commit message: Updated names
Parts:
- SW74: renamed from SW64; value Rctrl -> SW_Push
- renumbered D67 to D66, D66 to D67, SW65 to SW0, SW81 to SW100, Num1 to SW101, SW83 to SW102, Num2 to SW103, SW84 to SW104, `4 to SW14, SW14 to SW15, F1 to SW16, SW15 to SW17, SW16 to SW18, SW17 to SW19, SW18 to SW20, SW19 to SW21, SW20 to SW22, SW21 to SW23, SW22 to SW24, SW23 to SW25, SW24 to SW26, backspace1 to SW27, TAb1 to SW28, SW3 to SW29, F3 to SW30, SW26 to SW31, SW27 to SW32, SW28 to SW33, SW29 to SW34, SW30 to SW35, SW31 to SW36, SW32 to SW37, SW33 to SW38, SW34 to SW39, SW35 to SW40, \|1 to SW41, caps1 to SW42, SW37 to SW43, F4 to SW44, SW38 to SW45, SW39 to SW46, SW40 to SW47, SW41 to SW48, SW42 to SW49, SW43 to SW50, SW44 to SW51, SW45 to SW52, SW46 to SW53, enter1 to SW54, Lshift1 to SW55, SW48 to SW56, F5 to SW57, SW49 to SW58, SW50 to SW59, SW51 to SW60, SW52 to SW61, SW53 to SW62, SW54 to SW63, SW55 to SW64, SW56 to SW65, Rshift1 to SW66, SW57 to SW67, F6 to SW68, SW59 to SW69, Space1 to SW70, SW61 to SW71, SW62 to SW72, SW63 to SW73, SW25 to SW75, SW36 to SW76, SW47 to SW77, SW58 to SW78, SW60 to SW79, SW66 to SW81, SW67 to SW82, SW68 to SW83, F7 to SW84, SW70 to SW85, SW71 to SW86, SW72 to SW87, F8 to SW88, SW74 to SW89, F9 to SW90, F10 to SW91, SW69 to SW92, SW73 to SW93, SW75 to SW94, NumEnter1 to SW95, SW77 to SW96, SW78 to SW97, SW79 to SW98, SW80 to SW99

Commit message: updated some documentation
Parts:
- R1, R2, R3, R4: value R -> 2k
Changed lines of the file:
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@@
 			)
 		)
-		(property "Value" "R"
+		(property "Value" "2k"
 			(at 3.81 1.92 0)
 			(layer "F.Fab")
@@
 			)
 		)
-		(property "Value" "R"
+		(property "Value" "2k"
 			(at 3.81 1.92 0)
 			(layer "F.Fab")
@@
 			)
 		)
-		(property "Value" "R"
+		(property "Value" "2k"
 			(at 3.81 1.92 0)
 			(layer "F.Fab")
@@
 			)
 		)
-		(property "Value" "R"
+		(property "Value" "2k"
 			(at 3.81 1.92 0)
 			(layer "F.Fab")
